Commit message: Added a bunch of things

File: warnie/robot_extras/husky/husky_camera.urdf.xacro (robot description, xacro)
@@ -8,4 +8,24 @@
     <parent link="base_link" />
     <child link="2d_camera_link" />
+  </joint>
+  <!-- bumper box -->
+  <link name="bumper_box_link">
+    <visual>
+      <origin xyz="0 0 0" rpy="0 0 0" />
+      <geometry>
+        <mesh filename="package://warnie/robot_extras/husky/husky_bumper_box/husky_bumper_box.stl" />
+      </geometry>
+    </visual>
+    <collision>
+      <origin xyz="0 0 0" rpy="0 0 0" />
+      <geometry>
+        <mesh filename="package://warnie/robot_extras/husky/husky_bumper_box/husky_bumper_box.stl" />
+      </geometry>
+    </collision>
+  </link>
+  <joint name="bumper_box_joint" type="fixed">
+    <origin xyz="0 0 0.05" rpy="0 0 0" />
+    <parent link="base_link" />
+    <child link="bumper_box_link" />
   </joint>
   <!-- camera -->

Commit message: Created biased traps

File: warnie/robot_extras/husky/husky_camera.urdf.xacro (robot description, xacro)
@@ -29,4 +29,21 @@
     <child link="bumper_box_link" />
   </joint>
+  <!--link name="fov_wall_link">
+    <visual>
+      <origin xyz="0 0 0" rpy="0 0 0" />
+      <geometry>
+        <mesh filename="package://warnie/robot_extras/husky/fov_wall.stl" />
+      </geometry>
+      <material name="TransparentGrey"/>
+    </visual>
+  </link>
+  <gazebo reference="fov_wall_link">
+   <material>Gazebo/TransparentGrey</material>
+  </gazebo>
+  <joint name="fov_wall_joint" type="fixed">
+    <origin xyz="10 0 0" rpy="0 0 0" />
+    <parent link="base_link" />
+    <child link="fov_wall_link" />
+  </joint-->
   <!-- camera -->
   <gazebo reference="2d_camera_link">
@@ -42,5 +59,5 @@
         <clip>
           <near>0.02</near>
-          <far>300</far>
+          <far>200</far>
         </clip>
       </camera>

Commit message: Added R script for creating plots

File: warnie/robot_extras/husky/husky_camera.urdf.xacro (robot description, xacro)
@@ -11,10 +11,10 @@
   <!-- bumper box -->
   <link name="bumper_box_link">
-    <visual>
-      <origin xyz="0 0 0" rpy="0 0 0" />
-      <geometry>
-        <mesh filename="package://warnie/robot_extras/husky/husky_bumper_box/husky_bumper_box.stl" />
-      </geometry>
-    </visual>
+<!--    <visual>-->
+<!--      <origin xyz="0 0 0" rpy="0 0 0" />-->
+<!--      <geometry>-->
+<!--        <mesh filename="package://warnie/robot_extras/husky/husky_bumper_box/husky_bumper_box.stl" />-->
+<!--      </geometry>-->
+<!--    </visual>-->
     <collision>
       <origin xyz="0 0 0" rpy="0 0 0" />
